Commit message: Telop core add v2.6.6

File: linkertelopsdk/ros1/example/assets/robots/hands/linker_hand/l10_left/linkerhand_l10_left.urdf (robot description, URDF)
Before this commit: robot linkerhand_l10_7_left.urdf, 21 links, 20 joints
Joints:
- joint pinky_mcp_roll: axis -0.99996 0 0.0087265 -> 0.99996 0 0.0087265; limit lower=0 upper=0.3489 effort=100 velocity=1 -> lower=-0.3489 upper=0 effort=100 velocity=1
- joint ring_mcp_roll: axis -0.99996 0 0.0087265 -> 0.99996 0 0.0087265; limit lower=0 upper=0.2181 effort=100 velocity=1 -> lower=-0.2181 upper=0 effort=100 velocity=1

File: linkertelopsdk/ros1/example/assets/robots/hands/linker_hand/l10_right/linkerhand_l10_right.urdf (robot description, URDF)
Before this commit: robot linkerhand_l10_7_right.urdf, 21 links, 20 joints
Joints:
- joint index_mcp_roll: axis -0.99996 0 0.0087265 -> 0.99996 0 0.0087265; limit lower=0 upper=0.2181 effort=100 velocity=1 -> lower=-0.2181 upper=0 effort=100 velocity=1
