Commit message: update ros2 to v2.6.6

File: linkertelopsdk/ros2/src/linkerhand_retarget/resource/assets/robots/hands/linker_hand/l25_right/linkerhand_l25_right.urdf (robot description, URDF)
Before this commit: robot linkerhand_l25_right, 27 links, 26 joints
Links:
- removed link base_link
- removed link index_link0
- removed link index_link1
- removed link index_link2
- removed link index_link3
- removed link index_link4
- removed link little_link0
- removed link little_link1
- removed link little_link2
- removed link little_link3
- removed link little_link4
- removed link middle_link0
- removed link middle_link1
- removed link middle_link2
- removed link middle_link3
- removed link middle_link4
- removed link ring_link0
- removed link ring_link1
- removed link ring_link2
- removed link ring_link3
- removed link ring_link4
- removed link trumb_link0
- removed link trumb_link1
- removed link trumb_link2
- removed link trumb_link3
- removed link trumb_link4
- removed link trumb_link5
- added link hand_base_link, mass 0.077055; collision mesh filename=meshes/hand_base_link.STL; visual mesh filename=meshes/hand_base_link.STL
- added link index_distal, mass 9.6249E-06; collision mesh filename=meshes/index_distal.STL; visual mesh filename=meshes/index_distal.STL
- added link index_metacarpals, mass 0.0029534; collision mesh filename=meshes/index_metacarpals.STL; visual mesh filename=meshes/index_metacarpals.STL
- added link index_middle, mass 4.0832E-06; collision mesh filename=meshes/index_middle.STL; visual mesh filename=meshes/index_middle.STL
- added link index_proximal, mass 0.0093494; collision mesh filename=meshes/index_proximal.STL; visual mesh filename=meshes/index_proximal.STL
- added link middle_distal, mass 9.6249E-06; collision mesh filename=meshes/middle_distal.STL; visual mesh filename=meshes/middle_distal.STL
- added link middle_metacarpals, mass 0.0029534; collision mesh filename=meshes/middle_metacarpals.STL; visual mesh filename=meshes/middle_metacarpals.STL
- added link middle_middle, mass 4.0832E-06; collision mesh filename=meshes/middle_middle.STL; visual mesh filename=meshes/middle_middle.STL
- added link middle_proximal, mass 0.0093494; collision mesh filename=meshes/middle_proximal.STL; visual mesh filename=meshes/middle_proximal.STL
- added link pinky_distal, mass 9.6249E-06; collision mesh filename=meshes/pinky_distal.STL; visual mesh filename=meshes/pinky_distal.STL
- added link pinky_metacarpals, mass 0.0029534; collision mesh filename=meshes/pinky_metacarpals.STL; visual mesh filename=meshes/pinky_metacarpals.STL
- added link pinky_middle, mass 4.0832E-06; collision mesh filename=meshes/pinky_middle.STL; visual mesh filename=meshes/pinky_middle.STL
- added link pinky_proximal, mass 0.0093494; collision mesh filename=meshes/pinky_proximal.STL; visual mesh filename=meshes/pinky_proximal.STL
- added link ring_distal, mass 9.6249E-06; collision mesh filename=meshes/ring_distal.STL; visual mesh filename=meshes/ring_distal.STL
- added link ring_metacarpals, mass 0.0029534; collision mesh filename=meshes/ring_metacarpals.STL; visual mesh filename=meshes/ring_metacarpals.STL
- added link ring_middle, mass 4.0832E-06; collision mesh filename=meshes/ring_middle.STL; visual mesh filename=meshes/ring_middle.STL
- added link ring_proximal, mass 0.0093494; collision mesh filename=meshes/ring_proximal.STL; visual mesh filename=meshes/ring_proximal.STL
- added link thumb_distal, mass 4.7112E-06; collision mesh filename=meshes/thumb_distal.STL; visual mesh filename=meshes/thumb_distal.STL
- added link thumb_metacarpals, mass 0.019929; collision mesh filename=meshes/thumb_metacarpals.STL; visual mesh filename=meshes/thumb_metacarpals.STL
- added link thumb_metacarpals_base1, mass 0.010336; collision mesh filename=meshes/thumb_metacarpals_base1.STL; visual mesh filename=meshes/thumb_metacarpals_base1.STL
- added link thumb_metacarpals_base2, mass 0.002032; collision mesh filename=meshes/thumb_metacarpals_base2.STL; visual mesh filename=meshes/thumb_metacarpals_base2.STL
- added link thumb_proximal, mass 0.0061014; collision mesh filename=meshes/thumb_proximal.STL; visual mesh filename=meshes/thumb_proximal.STL
Joints:
- removed joint index_joint0
- removed joint index_joint1
- removed joint index_joint2
- removed joint index_joint3
- removed joint index_joint4
- removed joint little_joint0
- removed joint little_joint1
- removed joint little_joint2
- removed joint little_joint3
- removed joint little_joint4
- removed joint middle_joint0
- removed joint middle_joint1
- removed joint middle_joint2
- removed joint middle_joint3
- removed joint middle_joint4
- removed joint ring_joint0
- removed joint ring_joint1
- removed joint ring_joint2
- removed joint ring_joint3
- removed joint ring_joint4
- removed joint trumb_joint0
- removed joint trumb_joint1
- removed joint trumb_joint2
- removed joint trumb_joint3
- removed joint trumb_joint4
- removed joint trumb_joint5
- added joint index_dip: type revolute, parent index_middle, child index_distal, origin xyz=0.00099206 -0.00025106 0.044322 rpy=0 0 0, axis 0 1 0, limit lower=0 upper=1.78 effort=0 velocity=0
- added joint index_mcp_pitch: type revolute, parent index_metacarpals, child index_proximal, origin xyz=0.0068598 -0.00010189 0.018075 rpy=0 0 0, axis 0 0.99998 -0.0056645, limit lower=0 upper=1.68 effort=0 velocity=0
- added joint index_mcp_roll: type revolute, parent hand_base_link, child index_metacarpals, origin xyz=0.0014984 0.032141 0.13508 rpy=0 0 0, axis 1 0 0, limit lower=-0.24 upper=0.24 effort=0 velocity=0
- added joint index_pip: type revolute, parent index_proximal, child index_middle, origin xyz=-0.0001598 -0.00024924 0.043999 rpy=0 0 0, axis 0 0.99998 -0.0056645, limit lower=0 upper=1.27 effort=0 velocity=0
- added joint middle_dip: type revolute, parent middle_middle, child middle_distal, origin xyz=0.00099206 -0.00025106 0.044322 rpy=0 0 0, axis 0 1 0, limit lower=0 upper=1.78 effort=0 velocity=0
- added joint middle_mcp_pitch: type revolute, parent middle_metacarpals, child middle_proximal, origin xyz=0.0068598 -0.00010189 0.018075 rpy=0 0 0, axis 0 0.99998 -0.0056645, limit lower=0 upper=1.68 effort=0 velocity=0
- added joint middle_mcp_roll: type revolute, parent hand_base_link, child middle_metacarpals, origin xyz=0.0014985 0.0099581 0.14231 rpy=0 0 0, axis 1 0 0, limit lower=-0.24 upper=0.24 effort=0 velocity=0
- added joint middle_pip: type revolute, parent middle_proximal, child middle_middle, origin xyz=-0.0001598 -0.00024924 0.043999 rpy=0 0 0, axis 0 0.99998 -0.0056645, limit lower=0 upper=1.27 effort=0 velocity=0
- added joint pinky_dip: type revolute, parent pinky_middle, child pinky_distal, origin xyz=0.00099206 -0.00025106 0.044322 rpy=0 0 0, axis 0 1 0, limit lower=0 upper=1.78 effort=0 velocity=0
- added joint pinky_mcp_pitch: type revolute, parent pinky_metacarpals, child pinky_proximal, origin xyz=0.0068598 -0.00010189 0.018075 rpy=0 0 0, axis 0 0.99998 -0.0056645, limit lower=0 upper=1.68 effort=0 velocity=0
- added joint pinky_mcp_roll: type revolute, parent hand_base_link, child pinky_metacarpals, origin xyz=0.0014989 -0.033485 0.1194 rpy=0 0 0, axis 1 0 0, limit lower=-0.24 upper=0.24 effort=0 velocity=0
- added joint pinky_pip: type revolute, parent pinky_proximal, child pinky_middle, origin xyz=-0.0001598 -0.00024924 0.043999 rpy=0 0 0, axis 0 0.99998 -0.0056645, limit lower=0 upper=1.27 effort=0 velocity=0
- added joint ring_dip: type revolute, parent ring_middle, child ring_distal, origin xyz=0.00099206 -0.00025106 0.044322 rpy=0 0 0, axis 0 1 0, limit lower=0 upper=1.78 effort=0 velocity=0
- added joint ring_mcp_pitch: type revolute, parent ring_metacarpals, child ring_proximal, origin xyz=0.0068598 -0.00010189 0.018075 rpy=0 0 0, axis 0 0.99998 -0.0056645, limit lower=0 upper=1.68 effort=0 velocity=0
- added joint ring_mcp_roll: type revolute, parent hand_base_link, child ring_metacarpals, origin xyz=0.0014987 -0.011555 0.13457 rpy=0 0 0, axis 1 0 0, limit lower=-0.24 upper=0.24 effort=0 velocity=0
- added joint ring_pip: type revolute, parent ring_proximal, child ring_middle, origin xyz=-0.0001598 -0.00024924 0.043999 rpy=0 0 0, axis 0 0.99998 -0.0056645, limit lower=0 upper=1.27 effort=0 velocity=0
- added joint thumb_cmc_pitch: type revolute, parent thumb_metacarpals_base2, child thumb_metacarpals, origin xyz=0.006883 0.014309 0.0015936 rpy=0 0 0, axis 1 0 0, limit lower=0 upper=1.59 effort=0 velocity=0
- added joint thumb_cmc_roll: type revolute, parent hand_base_link, child thumb_metacarpals_base1, origin xyz=-0.016602 0.001612 0.071287 rpy=0 0 0, axis 1 0 0, limit lower=-0.46 upper=0.61 effort=0 velocity=0
- added joint thumb_cmc_yaw: type revolute, parent thumb_metacarpals_base1, child thumb_metacarpals_base2, origin xyz=0.04625 0.0083829 4.7486E-05 rpy=0 0 0, axis 0 0.0056645 -0.99998, limit lower=0 upper=1.57 effort=0 velocity=0
- added joint thumb_ip: type revolute, parent thumb_proximal, child thumb_distal, origin xyz=0 0.046252 -0.0020512 rpy=0 0 0, axis 1 0 0, limit lower=0 upper=1.78 effort=0 velocity=0
- added joint thumb_mcp: type revolute, parent thumb_metacarpals, child thumb_proximal, origin xyz=0 0.034264 -0.0037526 rpy=0 0 0, axis 1 0 0, limit lower=0- upper=1.59 effort=0 velocity=0
